File: Cart top solution/CTS Version 2.sch (EAGLE design)
At the start: 18 parts, among them J1 RASPBERRYPI-40-PIN-GPIO_PTH_N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, T2 2N2222, U1 RASPBERRY_PI_40SMD, X1 CON-WAGO_740_740-102, X2 CON-WAGO_740_740-102

Commit message: 2 sided board
Parts:
- removed CONVETER2: DC-DC-STEP-DOWN-MP1584, GHIdiy-modules:DC-DC-STEP-DOWN-MP1584
- removed POWER_JACK: (no value), con-jack:JACK-PLUG0
- removed R1: (no value), adafruit:R-US_0207/10
- removed R2, R3, R4, R5, R6: (no value), resistor:R-EU_0204/7
- removed X2: CON-WAGO_740_740-102, Termnal block:CON-WAGO_740_740-102
- added POWER_IN_12V: Power in (12V), Termnal block:CON-WAGO_740_740-102
- added R10, R11, R12, R7, R8, R9: 1k, SparkFun-Resistors:1KOHM-HORIZ-1/4W-5%
- added U$3: RTC-DS3231-AT24C32, GHIdiy-modulesRTC:RTC-DS3231-AT24C32
- U$2: value RTC-DS3231-AT24C32 -> DC-DC-STEP-DOWN-MP1584; device GHIdiy-modules:RTC-DS3231-AT24C32 -> GHIdiy-modulesRTC:DC-DC-STEP-DOWN-MP1584
- renumbered X1 to TO_PRINTER_19V
Connections:
- removed net N$16: R2.2, R3.1
- removed net N$17: R3.2, R4.1
- removed net N$18: R4.2, R5.1
- removed net N$21: R2.1, X2.P1
- new net N$15: R10.1, R9.2
- new net N$20: R10.2, R11.1
- net GND: now also CONVETER1.IN-, POWER_IN_12V.P2, R12.2, T2.E, U$2.IN-.1, U$2.OUT-.1, U$3.GND.1; no longer CONVETER2.OUT-.1, R6.2, U$2.GND.1, X2.P2
- net N$1: now also POWER_IN_12V.P1, R8.1, U$2.IN+.2; no longer CONVETER2.IN+.2, POWER_JACK.3
- net N$11: now also R7.1; no longer R1.1
- net N$19: now also R11.2, R12.1; no longer R5.2, R6.1
- net N$2: now also U$3.SDA.1; no longer U$2.SDA.1
- net N$5: now also R8.2, R9.1; no longer CONVETER1.IN-, CONVETER2.IN-.1, POWER_JACK.1, T2.E
- net N$50: now also U$3.SCL.1; no longer U$2.SCL.1
- net N$6: now also J1.MISO; no longer J1.GP19
- net N$7: now also R7.2; no longer R1.2
- net N$9: now also J1.MOSI; no longer J1.GP20
- net VCC: now also U$2.OUT+.2, U$3.VCC.1; no longer CONVETER2.OUT+.2, U$2.VCC.1
Other:
- moved on the sheet: U1
